File: bbf-audio_out/bbf-audio_out_v1.kicad_pcb (KiCad board)
At the start: 2 copper layers, 21.6 x 52.1 mm, 11 parts, among them IC1 TL072P, J5 MONOSWSLIM

Commit message: Update Readme.md
Add Logos
Update attribution
Parts:
- added G***: LOGO, _NTSFootprints:schenktronics.com_OSHW_Logo_6x6mm, F.Cu at (142.0, 128.0)
Other:
- board text added: "originally by: Émilie Gillet"
- board text removed: "Émilie Gillet"
