File: bbf-eurojacks/bbf-eurojacks_v1.kicad_pcb (KiCad board)
At the start: 2 copper layers, 16.5 x 52.1 mm, 7 parts, among them J1 1502_03SLOTTED, J2 1502_03SLOTTED, J3 1502_03SLOTTED, J4 1502_03SLOTTED

Commit message: Update jack footprint
Routing:
- net Net-(J2-Pad2): track 6.08 -> 7.93 mm
- net Net-(J4-Pad2): track 9.99 -> 10.5 mm

Commit message: Update Readme.md
Add Logos
Update attribution
Parts:
- added G***: LOGO, _NTSFootprints:schenktronics.com_OSHW_Logo_6x6mm, F.Cu at (143.0, 119.5)
Other:
- board text added: "originally by: Émilie Gillet"
- board text removed: "Émilie Gillet"
