File: bbf-europower/bbf-europower.kicad_pcb (KiCad board)
At the start: 2 copper layers, 16.5 x 52.1 mm, 12 parts, among them J1 CON_HEADER_2X05-PTH, J2 CON_HEADER_2X05-PTH

Commit message: Update Readme.md
Add Logos
Update attribution
Parts:
- added G***: LOGO, _NTSFootprints:schenktronics.com_OSHW_Logo_6x6mm, F.Cu at (153.5, 122.0)
Other:
- board text added: "Originally by: G. Johnson"
- board text removed: "G. Johnson"
