File: bbf-pots/bbf-pots_v1.kicad_pcb (KiCad board)
At the start: 2 copper layers, 16.5 x 52.1 mm, 6 parts

Commit message: Update Readme.md
Add Logos
Update attribution
Parts:
- added G***: LOGO, _NTSFootprints:schenktronics.com_OSHW_Logo_6x6mm, F.Cu at (142.8, 123.2)
Other:
- board text added: "Originally by: Émilie Gillet"
- board text removed: "Émilie Gillet"
