File: bbf-supply/bbf-supply_v1.kicad_pcb (KiCad board)
At the start: 2 copper layers, 21.6 x 52.1 mm, 16 parts, among them IC1 780X, IC2 LT1054, IC3 790X, J1 JACK-PLUG2

Commit message: Update Readme.md
Add Logos
Update attribution
Parts:
- added G***: LOGO, _NTSFootprints:schenktronics.com_OSHW_Logo_6x6mm, B.Cu at (143.8, 98.2)
Other:
- board text added: "Originally by: Émilie Gillet"
- board text removed: "Émilie Gillet"
