File: bbf-thonkjacks/bbf-thonkjacks.kicad_pcb (KiCad board)
At the start: 2 copper layers, 20.3 x 52.1 mm, 7 parts, among them J1 WQP-PJ301M-12_JACK, J2 WQP-PJ301M-12_JACK, J3 WQP-PJ301M-12_JACK, J4 WQP-PJ301M-12_JACK

Commit message: Update Readme.md
Add Logos
Update attribution
Parts:
- added G***: LOGO, _NTSFootprints:schenktronics.com_OSHW_Logo_6x6mm, F.Cu at (141.2, 120.2)
Other:
- board text added: "Originally By: G. Johnson"
- board text removed: "G. Johnson"
