File: bbf-buffer/bbf-midi/bbf-midi.sch (KiCad schematic (older format))
At the start: 17 parts, among them J1 Conn_02x05_Odd_Even, J2 Conn_02x05_Odd_Even, J3 DIN-5_180degree, J4 DIN-5_180degree, J5 Conn_01x03, U1 TLV1117-50, U2 6N137

Commit message: Update midi friend to 3.3v, including RX buffer.
Parts:
- removed U2: 6N137, Package_DIP:DIP-8_W7.62mm_Socket, symbol Isolator:6N137
- added C5: 100n, Capacitor_THT:C_Disc_D3.0mm_W2.0mm_P2.50mm, symbol Device:C_Small
- added Q1: 2N3904, Package_TO_SOT_THT:TO-92_Inline, symbol Transistor_BJT:2N3904
- added R5: 1K, Resistor_THT:R_Axial_DIN0207_L6.3mm_D2.5mm_P7.62mm_Horizontal, symbol Device:R_Small
- added U2: H11L1, Package_DIP:DIP-6_W7.62mm_Socket, symbol Isolator:H11L1
- C1, C2: footprint Capacitor_THT:CP_Radial_D6.3mm_P2.50mm -> Capacitor_THT:CP_Radial_D5.0mm_P2.50mm
- R1: value 220 -> 33
- R3: value 220 -> 10
- U1: value TLV1117-50 -> TLV1117-33; symbol Regulator_Linear:TLV1117-50 -> Regulator_Linear:TLV1117-33
- renumbered R5 to R6
Connections:
- net GND: now also C5.2, U2.5; no longer U1.1 (GND)
- net VCC: now also C5.1, R5.2, U2.6
- net at D1.2 (A), J3.5: now also U2.2
- net at D1.1 (K), R2.1: now also U2.1
- net at J5.2 (Pin_2), R6.1: now also U2.4
- net at R4.1: now also R1.2, Q1.3 (C)
- net at J5.3 (Pin_3): now also Q1.1 (E); no longer R1.2
- new net: Q1.2 (B), R5.1
- no-connect marks 5 -> 4
Other:
- moved on the sheet: C3, J4, R1, R3, R6, U1
